File: gsm.sch (EAGLE design)
At the start: 78 parts, among them J3 U.FL, J4 AVR_SPI_PROG_3X2OFFSET_PADS, J5 U.FL, Q1 600mA/40V, Q2 35A/25V/8.5mΩ, Q3 FDN360P, Q4 FDN360P, U1 LTC4056ETS8-4_2, U2 R-78E5.0-1.0, U3 LM2623MM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

Commit message: Before removing ttl compatibility with a direct connection
Parts:
- removed C16: 0.1uF, SparkFun-Capacitors:0.33UF/330NF-0805-50V-10%
- removed LED2: (no value), led:LEDCHIPLED_0805
- removed R23: 1k, SparkFun-Resistors:0.3OHM-0805-1/8W-1%
- R13: value 220 -> 10k
- U4, U8: SPICEPREFIX (none) -> X
Connections:
- removed net N$11: R23.1, U8.UART_RI
- removed net N$14: LED2.A, R23.2
- net +3V3: now also R13.2; no longer C16.1
- net GND: no longer LED2.C, R13.1
- net SIMVCC: now also U8.VSIM
- net SIM_POWKEY: now also R13.1; no longer C16.2, R13.2
Other:
- moved on the sheet: R13, R18
